File: Verakey.kicad_sch (KiCad schematic)
At the start: 19 parts, among them J1 Conn_01x04_Pin, J2 USB_C_Receptacle_USB2.0_16P, U1 STM32L432KBUx, U2 ATECC608A-MAHDA, U3 USBLC6-2SC6, U4 TLV75533PDBV

Commit message: First release
Parts:
- added C7: 100nF, Capacitor_SMD:C_0504_1310Metric, symbol Device:C_Small_US
- added R5, R6, R7, R8: 4.7k, Resistor_SMD:R_0402_1005Metric, symbol Device:R_Small_US
- added R9: 10k, Resistor_SMD:R_0603_1608Metric, symbol Device:R_Small_US
- added TP1: TestPoint_2Pole, Connector_PinHeader_1.00mm:PinHeader_1x02_P1.00mm_Vertical, symbol Connector:TestPoint_2Pole
- C4: value 100uF -> 10uF
- C5, C6: footprint Capacitor_SMD:C_0402_1005Metric -> Capacitor_SMD:C_0603_1608Metric
Connections:
- net +3.3V: now also R5.1, R6.1, R7.1, R8.1, R9.1
- net GND: now also C7.1, TP1.1
- net PA7: now also R5.2
- net PB4: now also R6.2
- net PB6: now also R8.2
- net PB7: now also R7.2
- net at U1.4 (NRST): now also C7.2, R9.2, TP1.2
